File: Williams System 9 display.kicad_pcb (KiCad board)
At the start: 4 copper layers, 96.3 x 53.2 mm, 30 parts, among them J101 Conn_01x02, J102 Conn_01x08, J103 Conn_01x08, J104 Conn_01x03, J105 Conn_01x04, J106 Conn_01x04, U101 74HC148, U102 74LV08A, U103 Pico, U104 74HC148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

Commit message: Address the remaining ERC violations
Parts:
- U107: footprint Package_TO_SOT_SMD_AKL:SOT-363_SC-70-6_BigPads -> Package_TO_SOT_SMD_AKL:SOT-363_SC-70-6_Handsoldering
Changed lines of the file:
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@@
     )
   )
-  (footprint "Package_TO_SOT_SMD_AKL:SOT-363_SC-70-6_BigPads" (layer "F.Cu")
+  (footprint "Package_TO_SOT_SMD_AKL:SOT-363_SC-70-6_Handsoldering" (layer "F.Cu")
     (at 238 55 180)
     (descr "SOT-363, SC-70-6, Handsoldering, Alternate KiCad Library")
@@
     (property "ki_description" "5.5-V, 1.5-A 79-mΩ, Low IQ Ideal Diode With Input Polarity Protection")
     (attr smd)
-    (fp_text reference "U107" (at 0 -2.23 180) (layer "F.SilkS") hide
+    (fp_text reference "U107" (at 0 -2 180) (layer "F.SilkS") hide
         (effects (font (size 1 1) (thickness 0.15)))
     )
-    (fp_text value "LM66100" (at 0 2) (layer "F.Fab") hide
+    (fp_text value "LM66100" (at 0 2) (layer "F.Fab")
         (effects (font (size 1 1) (thickness 0.15)))
     )
-    (fp_text user "${REFERENCE}" (at 0.3 0 270) (layer "F.Fab")
+    (fp_text user "${REFERENCE}" (at 0 0 270) (layer "F.Fab")
         (effects (font (size 0.5 0.5) (thickness 0.075)))
     )
-    (fp_line (start -2.5 -0.9) (end -2.5 1.5)
+    (fp_line (start -2.3495 -0.8255) (end -2.3495 1.27)
       (stroke (width 0.12) (type solid)) (layer "F.SilkS"))
-    (fp_line (start -2.5 1.5) (end 2.5 1.5)
+    (fp_line (start -2.3495 1.27) (end 2.3495 1.27)
       (stroke (width 0.12) (type solid)) (layer "F.SilkS"))
-    (fp_line (start 2.5 -1.5) (end -1.9 -1.5)
+    (fp_line (start 2.3495 -1.27) (end -1.905 -1.27)
       (stroke (width 0.12) (type solid)) (layer "F.SilkS"))
-    (fp_line (start 2.5 1.5) (end 2.5 -1.5)
+    (fp_line (start 2.3495 1.27) (end 2.3495 -1.27)
       (stroke (width 0.12) (type solid)) (layer "F.SilkS"))
-    (fp_circle (center -2.3 -1.3) (end -2.2365 -1.3)
+    (fp_circle (center -2.2225 -1.143) (end -2.159 -1.143)
       (stroke (width 0.2) (type solid)) (fill none) (layer "F.SilkS"))
     (fp_line (start -2.4 -1.4) (end -2.4 1.4)
@@
     (fp_line (start 2.4 1.4) (end 2.4 -1.4)
       (stroke (width 0.05) (type solid)) (layer "F.CrtYd"))
-    (fp_line (start -1.15 -0.8) (end -1.15 -0.5)
+    (fp_line (start -0.675 -0.6) (end -0.675 1.1)
       (stroke (width 0.1) (type solid)) (layer "F.Fab"))
-    (fp_line (start -1.15 -0.8) (end -0.7 -0.8)
+    (fp_line (start -0.175 -1.1) (end -0.675 -0.6)
       (stroke (width 0.1) (type solid)) (layer "F.Fab"))
-    (fp_line (start -1.15 -0.5) (end -0.7 -0.5)
-      (stroke (width 0.1) (type solid)) (layer "F.Fab"))
-    (fp_line (start -1.15 -0.15) (end -1.15 0.15)
-      (stroke (width 0.1) (type solid)) (layer "F.Fab"))
-    (fp_line (start -1.15 -0.15) (end -0.7 -0.15)
-      (stroke (width 0.1) (type solid)) (layer "F.Fab"))
-    (fp_line (start -1.15 0.15) (end -0.7 0.15)
-      (stroke (width 0.1) (type solid)) (layer "F.Fab"))
-    (fp_line (start -1.15 0.5) (end -1.15 0.8)
-      (stroke (width 0.1) (type solid)) (layer "F.Fab"))
-    (fp_line (start -1.15 0.5) (end -0.7 0.5)
-      (stroke (width 0.1) (type solid)) (layer "F.Fab"))
-    (fp_line (start -1.15 0.8) (end -0.7 0.8)
-      (stroke (width 0.1) (type solid)) (layer "F.Fab"))
-    (fp_line (start -0.675 -1.1) (end -0.675 1.1)
-      (stroke (width 0.1) (type solid)) (layer "F.Fab"))
-    (fp_line (start 0.675 -1.1) (end -0.675 -1.1)
+    (fp_line (start 0.675 -1.1) (end -0.175 -1.1)
       (stroke (width 0.1) (type solid)) (layer "F.Fab"))
     (fp_line (start 0.675 -1.1) (end 0.675 1.1)
@@
     (fp_line (start 0.675 1.1) (end -0.675 1.1)
       (stroke (width 0.1) (type solid)) (layer "F.Fab"))
-    (fp_line (start 1.15 -0.8) (end 0.7 -0.8)
-      (stroke (width 0.1) (type solid)) (layer "F.Fab"))
-    (fp_line (start 1.15 -0.5) (end 0.7 -0.5)
-      (stroke (width 0.1) (type solid)) (layer "F.Fab"))
-    (fp_line (start 1.15 -0.5) (end 1.15 -0.8)
-      (stroke (width 0.1) (type solid)) (layer "F.Fab"))
-    (fp_line (start 1.15 -0.15) (end 0.7 -0.15)
-      (stroke (width 0.1) (type solid)) (layer "F.Fab"))
-    (fp_line (start 1.15 0.15) (end 0.7 0.15)
-      (stroke (width 0.1) (type solid)) (layer "F.Fab"))
-    (fp_line (start 1.15 0.15) (end 1.15 -0.15)
-      (stroke (width 0.1) (type solid)) (layer "F.Fab"))
-    (fp_line (start 1.15 0.5) (end 0.7 0.5)
-      (stroke (width 0.1) (type solid)) (layer "F.Fab"))
-    (fp_line (start 1.15 0.8) (end 0.7 0.8)
-      (stroke (width 0.1) (type solid)) (layer "F.Fab"))
-    (fp_line (start 1.15 0.8) (end 1.15 0.5)
-      (stroke (width 0.1) (type solid)) (layer "F.Fab"))
-    (fp_circle (center -0.25 -0.7) (end -0.15 -0.7)
-      (stroke (width 0.1) (type solid)) (fill solid) (layer "F.Fab"))
-    (pad "1" smd roundrect (at -1.33 -0.65 180) (size 1.5 0.4) (layers "F.Cu" "F.Paste" "F.Mask") (roundrect_rratio 0.25)
+    (pad "1" smd rect (at -1.33 -0.65 180) (size 1.5 0.4) (layers "F.Cu" "F.Paste" "F.Mask")
       (net 86 "/V_{IN}") (pinfunction "V_{IN}") (pintype "power_in"))
-    (pad "2" smd roundrect (at -1.33 0 180) (size 1.5 0.4) (layers "F.Cu" "F.Paste" "F.Mask") (roundrect_rratio 0.25)
+    (pad "2" smd rect (at -1.33 0 180) (size 1.5 0.4) (layers "F.Cu" "F.Paste" "F.Mask")
       (net 2 "GND") (pinfunction "GND") (pintype "power_in"))
-    (pad "3" smd roundrect (at -1.33 0.65 180) (size 1.5 0.4) (layers "F.Cu" "F.Paste" "F.Mask") (roundrect_rratio 0.25)
+    (pad "3" smd rect (at -1.33 0.65 180) (size 1.5 0.4) (layers "F.Cu" "F.Paste" "F.Mask")
       (net 2 "GND") (pinfunction "~{CE}") (pintype "input"))
-    (pad "4" smd roundrect (at 1.33 0.65 180) (size 1.5 0.4) (layers "F.Cu" "F.Paste" "F.Mask") (roundrect_rratio 0.25)
+    (pad "4" smd rect (at 1.33 0.65 180) (size 1.5 0.4) (layers "F.Cu" "F.Paste" "F.Mask")
       (net 87 "unconnected-(U107-N{slash}C-Pad4)") (pinfunction "N/C") (pintype "no_connect"))
-    (pad "5" smd roundrect (at 1.33 0 180) (size 1.5 0.4) (layers "F.Cu" "F.Paste" "F.Mask") (roundrect_rratio 0.25)
-      (net 2 "GND") (pinfunction "ST") (pintype "output"))
-    (pad "6" smd roundrect (at 1.33 -0.65 180) (size 1.5 0.4) (layers "F.Cu" "F.Paste" "F.Mask") (roundrect_rratio 0.25)
+    (pad "5" smd rect (at 1.33 0 180) (size 1.5 0.4) (layers "F.Cu" "F.Paste" "F.Mask")
+      (net 2 "GND") (pinfunction "ST_{NA}") (pintype "passive"))
+    (pad "6" smd rect (at 1.33 -0.65 180) (size 1.5 0.4) (layers "F.Cu" "F.Paste" "F.Mask")
       (net 1 "+5V") (pinfunction "V_{OUT}") (pintype "power_out"))
     (model "${KICAD6_3DMODEL_DIR}/Package_TO_SOT_SMD.3dshapes/SOT-363_SC-70-6.wrl"
